File: v2/design/Alarm2.kicad_pcb (KiCad board)
At the start: 2 copper layers, 58 x 41.5 mm, 19 parts, among them J1 10118193-0001LF, J2 AVR-ISP-6, SW1 SW_Push, SW2 SW_Push, SW3 SW_Push, SW4 SW_Push, U1 ATmega328P-PU, U2 DS1307+, Y1 32.768Khz

Commit message: Added V2 PCB
Parts:
- removed Y1: 32.768Khz, Crystal:Crystal_AT310_D3.0mm_L10.0mm_Horizontal
- U2: value DS1307+ -> DS3231MZ; footprint Package_DIP:DIP-8_W7.62mm -> Package_SO:SOIC-8_3.9x4.9mm_P1.27mm
- moved R6 21.9 mm to (145.3, 101.2)
- moved R5 16.2 mm to (142.0, 101.2)
- moved BT1 9.42 mm to (130.2, 104.1)
- moved U2 6.90 mm to (125.7, 92.1), turned to 0 degrees
Connections:
- J2 pad 1: Net-(D1-Pad7) -> Net-(J2-Pad1)
- J2 pad 3: Net-(D1-Pad8) -> Net-(J2-Pad3)
- J2 pad 4: Net-(D1-Pad6) -> Net-(J2-Pad4)
- U1 pad 14: Net-(D1-Pad3) -> Net-(U1-Pad14)
- U1 pad 15: Net-(D1-Pad4) -> Net-(U1-Pad15)
- U1 pad 16: Net-(D1-Pad5) -> Net-(U1-Pad16)
- U1 pad 17: Net-(D1-Pad6) -> Net-(J2-Pad4)
- U1 pad 18: Net-(D1-Pad7) -> Net-(J2-Pad1)
- U1 pad 19: Net-(D1-Pad8) -> Net-(J2-Pad3)
- U2 pad 2: Net-(U2-Pad2) -> Net-(C1-Pad1)
- U2 pad 3: Net-(BT1-Pad1) -> Net-(U2-Pad3)
- U2 pad 4: Net-(BT1-Pad2) -> Net-(U2-Pad4)
- U2 pad 5: Net-(R5-Pad2) -> Net-(BT1-Pad2)
- U2 pad 6: Net-(R6-Pad2) -> Net-(BT1-Pad1)
- U2 pad 7: Net-(U2-Pad7) -> Net-(R5-Pad2)
- U2 pad 8: Net-(C1-Pad1) -> Net-(R6-Pad2)
Routing:
- net Net-(C1-Pad1): track 161.0 -> 150.1 mm
- net Net-(U2-Pad1): track 4.40 -> 0.00 mm
- net Net-(U2-Pad2): track 4.37 -> 0.00 mm
- net Net-(BT1-Pad1): track 33.7 -> 30.0 mm
- net Net-(BT1-Pad2): track 119.0 -> 115.7 mm
- net Net-(R6-Pad2): track 32.2 -> 33.5 mm
